Commit message: IsaacSim 5.1, IsaacLab up-to-date 2025/11/08; modify urdf with removing inertial property

File: active_adaptation/g1_description/g1_29dof_rev_1_0.urdf (robot description, URDF)
Before this commit: robot g1_29dof_rev_1_0, 39 links, 38 joints
Links:
- link head_link: mass 1.036 -> None
- link left_rubber_hand: mass 0.170 -> None
- link logo_link: mass 0.001 -> None
- link pelvis_contour_link: mass 0.001 -> None
- link right_rubber_hand: mass 0.170 -> None
